Commit message: update urdf

File: src/piper_description/urdf/piper_no_gripper_description.urdf (robot description, URDF)
Before this commit: robot arm, 11 links, 10 joints
Links:
- removed link gripper_base
- removed link link7
- removed link link8
- removed link world
Joints:
- removed joint fixed_base_joint
- removed joint joint6_to_gripper_base
- removed joint joint7
- removed joint joint8
- joint joint6: limit lower=-2.0944 upper=2.0944 effort=100 velocity=3 -> lower=-2.0944 upper=2.0944 effort=100 velocity=5

File: src/piper_description/urdf/piper_no_gripper_description.xacro (robot description, xacro)
@@ -396,172 +396,5 @@
       upper="2.0944"
       effort="100"
-      velocity="3" />
-  </joint>
-  <link
-    name="gripper_base">
-    <inertial>
-      <origin
-        xyz="-0.000183807162235591 8.05033155577911E-05 0.0321436689908876"
-        rpy="0 0 0" />
-      <mass
-        value="0.145318531013916" />
-      <inertia
-        ixx="0.000101740348396288"
-        ixy="-1.43961090652723E-07"
-        ixz="-8.72352812740139E-08"
-        iyy="4.16518088621566E-05"
-        iyz="3.27712901952435E-08"
-        izz="0.000118691325723675" />
-    </inertial>
-    <visual>
-      <origin
-        xyz="0 0 0"
-        rpy="0 0 0" />
-      <geometry>
-        <mesh
-          filename="package://piper_description/meshes/gripper_base.STL" />
-      </geometry>
-      <material
-        name="">
-        <color
-          rgba="0.792156862745098 0.819607843137255 0.933333333333333 1" />
-      </material>
-    </visual>
-    <collision>
-      <origin
-        xyz="0 0 0"
-        rpy="0 0 0" />
-      <geometry>
-        <mesh
-          filename="package://piper_description/meshes/gripper_base.STL" />
-      </geometry>
-    </collision>
-  </link>
-  <joint
-    name="joint6_to_gripper_base"
-    type="fixed">
-    <origin
-      xyz="0 0 0"
-      rpy="0 0 0" />
-    <parent
-      link="link6" />
-    <child
-      link="gripper_base" />
-  </joint>
-  <link
-    name="link7">
-    <inertial>
-      <origin
-        xyz="0.00065123185041968 -0.0491929869131989 0.00972258769184025"
-        rpy="0 0 0" />
-      <mass
-        value="0.0303534920715906" />
-      <inertia
-        ixx="1.13870358991284E-05"
-        ixy="4.2853410993302E-07"
-        ixz="-6.45170690459141E-08"
-        iyy="6.26108891787743E-06"
-        iyz="1.5729036212893E-06"
-        izz="1.57822030592869E-05" />
-    </inertial>
-    <visual>
-      <origin
-        xyz="0 0 0"
-        rpy="0 0 0" />
-      <geometry>
-        <mesh
-          filename="package://piper_description/meshes/link7.STL" />
-      </geometry>
-      <material
-        name="">
-        <color
-          rgba="0.792156862745098 0.819607843137255 0.933333333333333 1" />
-      </material>
-    </visual>
-    <collision>
-      <origin
-        xyz="0 0 0"
-        rpy="0 0 0" />
-      <geometry>
-        <mesh
-          filename="package://piper_description/meshes/link7.STL" />
-      </geometry>
-    </collision>
-  </link>
-  <joint
-    name="joint7"
-    type="prismatic">
-    <origin
-      xyz="0 0 0.1358"
-      rpy="1.5708 0 0" />
-    <parent
-      link="gripper_base" />
-    <child
-      link="link7" />
-    <axis
-      xyz="0 0 1" />
-    <limit
-      lower="0"
-      upper="0.035"
-      effort="10"
-      velocity="1" />
-  </joint>
-  <link
-    name="link8">
-    <inertial>
-      <origin
-        xyz="0.000651231850419722 -0.0491929869131991 0.00972258769184024"
-        rpy="0 0 0" />
-      <mass
-        value="0.0303534920715904" />
-      <inertia
-        ixx="1.13870358991283E-05"
-        ixy="4.28534109932964E-07"
-        ixz="-6.45170690459078E-08"
-        iyy="6.26108891787742E-06"
-        iyz="1.57290362128933E-06"
-        izz="1.57822030592867E-05" />
-    </inertial>
-    <visual>
-      <origin
-        xyz="0 0 0"
-        rpy="0 0 0" />
-      <geometry>
-        <mesh
-          filename="package://piper_description/meshes/link8.STL" />
-      </geometry>
-      <material
-        name="">
-        <color
-          rgba="0.792156862745098 0.819607843137255 0.933333333333333 1" />
-      </material>
-    </visual>
-    <collision>
-      <origin
-        xyz="0 0 0"
-        rpy="0 0 0" />
-      <geometry>
-        <mesh
-          filename="package://piper_description/meshes/link8.STL" />
-      </geometry>
-    </collision>
-  </link>
-  <joint
-    name="joint8"
-    type="prismatic">
-    <origin
-      xyz="0 0 0.1358"
-      rpy="1.5708 0 -3.1416" />
-    <parent
-      link="gripper_base" />
-    <child
-      link="link8" />
-    <axis
-      xyz="0 0 -1" />
-    <limit
-      lower="-0.035"
-      upper="0"
-      effort="10"
-      velocity="1" />
+      velocity="5" />
   </joint>
 <!-- controller -->
@@ -584,6 +417,4 @@
   <xacro:transmission_block tran_name="tran5" joint_name="joint5" motor_name="motor5"/>
   <xacro:transmission_block tran_name="tran6" joint_name="joint6" motor_name="motor6"/>
-  <xacro:transmission_block tran_name="tran7" joint_name="joint7" motor_name="motor7"/>
-  <xacro:transmission_block tran_name="tran8" joint_name="joint8" motor_name="motor8"/>
 <!-- gazebo -->
   <gazebo>
@@ -593,30 +424,3 @@
     </plugin>
   </gazebo>
-  <!-- <gazebo reference="base_link">
-    <material>Gazebo/Black</material>
-  </gazebo>
-  <gazebo reference="link1">
-    <material>Gazebo/White</material>
-  </gazebo>
-  <gazebo reference="link2">
-    <material>Gazebo/White</material>
-  </gazebo>
-  <gazebo reference="link3">
-    <material>Gazebo/White</material>
-  </gazebo>
-  <gazebo reference="link4">
-    <material>Gazebo/Black</material>
-  </gazebo>
-  <gazebo reference="link5">
-    <material>Gazebo/White</material>
-  </gazebo>
-  <gazebo reference="link6">
-    <material>Gazebo/White</material>
-  </gazebo>
-  <gazebo reference="link7">
-    <material>Gazebo/Orange</material>
-  </gazebo>
-  <gazebo reference="link8">
-    <material>Gazebo/Orange</material>
-  </gazebo> -->
 </robot>
