Commit message: rqtで動的にtfの位置を変更してもmoveitで動作させることができた！

File: src/piper_description/urdf/piper_macro.xacro (robot description, xacro)
@@ -333,7 +333,7 @@
     <!-- RealSense D435i Camera -->
     <xacro:include filename="$(find realsense2_description)/urdf/_d435i.urdf.xacro" />
-    <xacro:sensor_d435i parent="gripper_base" name="camera" use_nominal_extrinsics="true" use_mesh="true">
-        <origin xyz="0.04 0 0.04" rpy="0 -1.57 3.14"/>
-    </xacro:sensor_d435i>
-  </xacro:macro>
+<xacro:sensor_d435i parent="gripper_base" name="camera" use_nominal_extrinsics="true">
+    <origin xyz="0.04 0 0.04" rpy="0 -1.57 3.14"/>
+</xacro:sensor_d435i>
+</xacro:macro>
 </robot>

Commit message: グリッパー開閉を単一ノードで確認 次はflexbe化

File: src/piper_description/urdf/piper_macro.xacro (robot description, xacro)
@@ -266,5 +266,5 @@
         <child link="link7" />
         <axis xyz="0 0 1" />
-        <limit lower="0" upper="0.035" effort="10" velocity="1" />
+        <limit lower="0" upper="0.099" effort="10" velocity="1" />
     </joint>
     <link name="link8">

Commit message: rvizの設定追記・realsenseのURDF位置を修正

File: src/piper_description/urdf/piper_macro.xacro (robot description, xacro)
@@ -335,5 +335,5 @@
     <xacro:include filename="$(find realsense2_description)/urdf/_d435i.urdf.xacro" />
 <xacro:sensor_d435i parent="gripper_base" name="camera" use_nominal_extrinsics="true">
-    <origin xyz="0.04 0 0.04" rpy="0 -1.57 3.14"/>
+    <origin xyz="-0.04 0.0 0.055" rpy="3.14 -1.6 3.14"/>
 </xacro:sensor_d435i>
 </xacro:macro>

Commit message: yolov8-segノードを追加

File: src/piper_description/urdf/piper_macro.xacro (robot description, xacro)
@@ -1,4 +1,6 @@
 <?xml version="1.0" encoding="utf-8"?>
 <robot xmlns:xacro="http://ros.org/wiki/xacro">
+  <xacro:property name="finger_length" value="0.04" />
+  <xacro:property name="joint_z_offset" value="0.1358" />
   <xacro:macro name="piper_robot">
     <!-- world -->
@@ -295,6 +297,12 @@
         <child link="link8" />
         <axis xyz="0 0 -1" />
-        <limit lower="-0.035" upper="0" effort="10" velocity="1" />
+        <limit lower="0" upper="0.099" effort="10" velocity="1" />
         <mimic joint="joint7" multiplier="1" offset="0" />
+    </joint>
+    <link name="tcp_link"/>
+    <joint name="tcp_joint" type="fixed">
+        <origin xyz="0 0 ${joint_z_offset + (finger_length / 2)}" rpy="0 0 0" />
+        <parent link="gripper_base" />
+        <child link="tcp_link" />
     </joint>
     <!-- Gazebo Materials -->

Commit message: グリッパのTF位置をパラチュー

File: src/piper_description/urdf/piper_macro.xacro (robot description, xacro)
@@ -1,6 +1,6 @@
 <?xml version="1.0" encoding="utf-8"?>
 <robot xmlns:xacro="http://ros.org/wiki/xacro">
-  <xacro:property name="finger_length" value="0.04" />
-  <xacro:property name="joint_z_offset" value="0.1358" />
+  <xacro:property name="finger_length" value="0.0" />
+  <xacro:property name="joint_z_offset" value="0.1058" />
   <xacro:macro name="piper_robot">
     <!-- world -->

Commit message: とりあえずpush

File: src/piper_description/urdf/piper_macro.xacro (robot description, xacro)
@@ -343,5 +343,5 @@
     <xacro:include filename="$(find realsense2_description)/urdf/_d435i.urdf.xacro" />
 <xacro:sensor_d435i parent="gripper_base" name="camera" use_nominal_extrinsics="true">
-    <origin xyz="-0.04 0.0 0.055" rpy="3.14 -1.6 3.14"/>
+    <origin xyz="-0.04 0.0 0.055" rpy="1.9154 1.5062 -1.0020"/>
 </xacro:sensor_d435i>
 </xacro:macro>

Commit message: realsenseカメラの位置姿勢がおよそ正しくなった。 まだわずかに傾いているので調整する。 一旦プッシュ

File: src/piper_description/urdf/piper_macro.xacro (robot description, xacro)
@@ -343,5 +343,5 @@
     <xacro:include filename="$(find realsense2_description)/urdf/_d435i.urdf.xacro" />
 <xacro:sensor_d435i parent="gripper_base" name="camera" use_nominal_extrinsics="true">
-    <origin xyz="-0.04 0.0 0.055" rpy="1.9154 1.5062 -1.0020"/>
+  <origin xyz="-0.04 0.0 0.055" rpy="2.9630 -1.5062 3.1396"/>
 </xacro:sensor_d435i>
 </xacro:macro>

Commit message: roll: 179.680 pitch: -89.994 yaw: -279.971 [deg]
でrealsenseカメラの位置を修正。

File: src/piper_description/urdf/piper_macro.xacro (robot description, xacro)
@@ -343,5 +343,6 @@
     <xacro:include filename="$(find realsense2_description)/urdf/_d435i.urdf.xacro" />
 <xacro:sensor_d435i parent="gripper_base" name="camera" use_nominal_extrinsics="true">
-  <origin xyz="-0.04 0.0 0.055" rpy="2.9630 -1.5062 3.1396"/>
+  <origin xyz="-0.04 0.0 0.055" rpy="3.1360 -1.5707 3.1421"/>
+  <!-- yaw 3.2586で -173.29 deg-->
 </xacro:sensor_d435i>
 </xacro:macro>

Commit message: カメラ姿勢キャリブレーション追加。 カメラ姿勢のせいでTF発行位置がずれる問題を修正。
キャリブレーション実行は
ros2 run piper rpy_calibiration_fixed   --ros-args   -p image_topic:=/camera/camera/color/image_raw   -p camera_info_topic:=/camera/camera/color/camera_info   -p base_frame:=base_link   -p parent_frame:=gripper_base   -p camera_link_frame:=camera_link   -p optical_frame:=camera_color_optical_frame   -p marker_id:=0   -p marker_length:=0.1

File: src/piper_description/urdf/piper_macro.xacro (robot description, xacro)
@@ -343,5 +343,5 @@
     <xacro:include filename="$(find realsense2_description)/urdf/_d435i.urdf.xacro" />
 <xacro:sensor_d435i parent="gripper_base" name="camera" use_nominal_extrinsics="true">
-  <origin xyz="-0.04 0.0 0.055" rpy="3.1360 -1.5707 3.1421"/>
+  <origin xyz="-0.04 0.0 0.055" rpy="0.033796 -1.458712 -0.038036"/>
   <!-- yaw 3.2586で -173.29 deg-->
 </xacro:sensor_d435i>
