Commit message: カチャカのURDF作成．ros1 --> ros2含め動作検証中

File: src/piper_description/urdf/piper_macro.xacro (robot description, xacro)
@@ -3,13 +3,22 @@
   <xacro:property name="finger_length" value="0.0" />
   <xacro:property name="joint_z_offset" value="0.1058" />
-  <xacro:macro name="piper_robot">
+  <xacro:macro name="piper_robot"
+               params="parent:='world'
+                       base_link_name:='base_link'
+                       base_joint_name:='fixed_base_joint'
+                       base_xyz:='0 0 0'
+                       base_rpy:='0 0 0'
+                       create_world:=true">
     <!-- world -->
-    <link name="world"/>
-    <joint name="fixed_base_joint" type="fixed">
-        <parent link="world"/>
-        <child link="base_link"/>
+    <xacro:if value="${create_world}">
+      <link name="world"/>
+    </xacro:if>
+    <joint name="${base_joint_name}" type="fixed">
+        <origin xyz="${base_xyz}" rpy="${base_rpy}"/>
+        <parent link="${parent}"/>
+        <child link="${base_link_name}"/>
     </joint>
     <!-- arm -->
-    <link name="base_link">
+    <link name="${base_link_name}">
         <inertial>
                 <origin xyz="-0.00473641164191482 2.56829134630247E-05 0.041451518036016" rpy="0 0 0" />
@@ -57,5 +66,5 @@
     <joint name="joint1" type="revolute">
         <origin xyz="0 0 0.123" rpy="0 0 0" />
-        <parent link="base_link" />
+        <parent link="${base_link_name}" />
         <child link="link1" />
         <axis xyz="0 0 1" />
@@ -307,5 +316,5 @@
     </joint>
     <!-- Gazebo Materials -->
-    <gazebo reference="base_link">
+    <gazebo reference="${base_link_name}">
       <material>Gazebo/White</material>
     </gazebo>
